File: kicad/pcb/bully.kicad_sch (KiCad schematic)
At the start: 29 parts, among them J1 SM04B-SRSS-TB(LF)(SN), J2 Conn_01x04, U1 W25Q128JVS, U3 RP2040, U4 XC6206PxxxMR-Regulator_Linear, Y1 12MHz

Commit message: Initial commit for colbully kbd.
Parts:
- removed J2: Conn_01x04, Connector_PinHeader_2.54mm:PinHeader_1x04_P2.54mm_Vertical, symbol Connector_Generic:Conn_01x04
- added J2: Conn_ARM_SWD_TagConnect_TC2030-NL, Connector:Tag-Connect_TC2030-IDC-NL_2x03_P1.27mm_Vertical, symbol Connector:Conn_ARM_SWD_TagConnect_TC2030-NL
Connections:
- net ENC_A is gone; now on net COL8: U3.3 (GPIO1)
- net ENC_B is gone; now on net COL7: U3.2 (GPIO0)
- net +3V3: now also J2.1 (VCC)
- net COL1: now also U3.18 (GPIO15); no longer U3.12 (GPIO9)
- net COL10: now also U3.5 (GPIO3); no longer U3.7 (GPIO5)
- net COL12: now also U3.7 (GPIO5); no longer U3.5 (GPIO3)
- net COL13: now also U3.8 (GPIO6); no longer U3.4 (GPIO2)
- net COL2: now also U3.17 (GPIO14); no longer U3.14 (GPIO11)
- net COL3: now also U3.16 (GPIO13); no longer U3.15 (GPIO12)
- net COL4: now also U3.15 (GPIO12); no longer U3.16 (GPIO13)
- net COL5: now also U3.14 (GPIO11); no longer U3.17 (GPIO14)
- net COL6: now also U3.12 (GPIO9); no longer U3.18 (GPIO15)
- net COL7: no longer U3.29 (GPIO18)
- net COL8: no longer U3.32 (GPIO21)
- net COL9: now also U3.4 (GPIO2); no longer U3.8 (GPIO6)
- net GND: now also J2.5 (GND)
- net SWCLK: now also J2.4 (SWCLK)
- net SWD: now also J2.2 (SWDIO)
- net ~{RESET}: now also J2.3 (~{RESET})
- new net GPIO18: U3.29 (GPIO18)
- new net GPIO21: U3.32 (GPIO21)
- no-connect marks 0 -> 3
Other:
- note removed: "SW debug breakout pads"
