File: kicad/pcb/key_matrix.kicad_sch (KiCad schematic)
At the start: 107 parts, among them SW1 SW_Push, SW10 SW_Push, SW11 SW_Push, SW12 SW_Push, SW13 SW_Push, SW14 SW_Push, SW15 SW_Push, SW16 SW_Push, SW17 SW_Push, SW18 SW_Push, SW19 SW_Push, SW2 SW_Push, SW20 SW_Push, SW21 SW_Push, SW22 SW_Push, SW23 SW_Push, SW24 SW_Push, SW25 SW_Push, SW26 SW_Push, SW27 SW_Push, SW28 SW_Push, SW29 SW_Push, SW3 SW_Push, SW30 SW_Push, SW31 SW_Push, SW32 SW_Push, SW33 SW_Push, SW34 SW_Push, SW35 SW_Push, SW36 SW_Push, SW37 SW_Push, SW38 SW_Push, SW39 SW_Push, SW4 SW_Push, SW40 SW_Push, SW41 SW_Push, SW42 SW_Push, SW43 SW_Push, SW44 SW_Push, SW45 SW_Push, SW5 SW_Push, SW54 RotaryEncoder_Switch, SW6 SW_Push, SW7 SW_Push, SW8 SW_Push, SW9 SW_Push

Commit message: Initial commit for colbully kbd.
Parts:
- removed C18, C19: 100n, Capacitor_SMD:C_0402_1005Metric, symbol Device:C
- removed D46, D47: LED, LED_SMD:LED_0805_2012Metric_Pad1.15x1.40mm_HandSolder, symbol Device:LED
- removed R2: 1k, Resistor_SMD:R_0805_2012Metric, symbol Device:R
- removed SW12: SW_Push, MX_Alps_Hybrid:MX-Alps-Hybrid-1U, symbol Switch:SW_Push
- removed SW14: SW_Push, MX_Solderable:MX-Solderable-1.25U, symbol Switch:SW_Push
- removed SW37: SW_Push, MX_Alps_Hybrid:MX-Alps-Hybrid-2.25U, symbol Switch:SW_Push
- removed SW38, SW40, SW43, SW45: SW_Push, MX_Alps_Hybrid:MX-Alps-Hybrid-1.25U, symbol Switch:SW_Push
- removed SW41, SW42: SW_Push, MX_Alps_Hybrid:MX-Alps-Hybrid-3U-ReversedStabilizers, symbol Switch:SW_Push
- removed SW54: RotaryEncoder_Switch, keebio:RotaryEncoder_EC11, symbol Device:RotaryEncoder_Switch
- added D26, D39, D44, D48, D52: 1N4148W, Diode_SMD:D_SOD-123, symbol Diode:1N4148W
- added D47: SK6812, colbully:SK6812-MINI-E, symbol LED:SK6812
- added SW26, SW46, SW50: SW_Push, colbully:CherryMX_18mm_MidHeight_Choc_Hotswap_rev5, symbol Switch:SW_Push
- SW1: footprint MX_Alps_Hybrid:MX-Alps-Hybrid-1.5U -> colbully:CherryMX_18mm_MidHeight_Choc_Hotswap_rev5
- SW10, SW11, SW12, SW13, SW15, SW16, SW17, SW18, SW19, SW2, SW20, SW21, SW22, SW23, SW24, SW3, SW4, SW5, SW6, SW7, SW8, SW9: footprint MX_Alps_Hybrid:MX-Alps-Hybrid-1U -> colbully:CherryMX_18mm_MidHeight_Choc_Hotswap_rev5
- SW14, SW25: footprint MX_Alps_Hybrid:MX-Alps-Hybrid-1.75U -> colbully:CherryMX_18mm_MidHeight_Choc_Hotswap_rev5
- SW27: renamed from SW26; footprint MX_Alps_Hybrid:MX-Alps-Hybrid-2.25U -> colbully:CherryMX_18mm_MidHeight_Choc_Hotswap_rev5
- SW28: renamed from SW27; footprint MX_Alps_Hybrid:MX-Alps-Hybrid-1U -> colbully:CherryMX_18mm_MidHeight_Choc_Hotswap_rev5
- SW29: renamed from SW28; footprint MX_Alps_Hybrid:MX-Alps-Hybrid-1U -> colbully:CherryMX_18mm_MidHeight_Choc_Hotswap_rev5
- SW30: renamed from SW29; footprint MX_Alps_Hybrid:MX-Alps-Hybrid-1U -> colbully:CherryMX_18mm_MidHeight_Choc_Hotswap_rev5
- SW31: renamed from SW30; footprint MX_Alps_Hybrid:MX-Alps-Hybrid-1U -> colbully:CherryMX_18mm_MidHeight_Choc_Hotswap_rev5
- SW32: renamed from SW31; footprint MX_Alps_Hybrid:MX-Alps-Hybrid-1U -> colbully:CherryMX_18mm_MidHeight_Choc_Hotswap_rev5
- SW33: renamed from SW32; footprint MX_Alps_Hybrid:MX-Alps-Hybrid-1U -> colbully:CherryMX_18mm_MidHeight_Choc_Hotswap_rev5
- SW34: renamed from SW33; footprint MX_Alps_Hybrid:MX-Alps-Hybrid-1U -> colbully:CherryMX_18mm_MidHeight_Choc_Hotswap_rev5
- SW35: renamed from SW34; footprint MX_Alps_Hybrid:MX-Alps-Hybrid-1U -> colbully:CherryMX_18mm_MidHeight_Choc_Hotswap_rev5
- SW36: renamed from SW35; footprint MX_Alps_Hybrid:MX-Alps-Hybrid-1U -> colbully:CherryMX_18mm_MidHeight_Choc_Hotswap_rev5
- SW37: renamed from SW36; footprint MX_Alps_Hybrid:MX-Alps-Hybrid-1U -> colbully:CherryMX_18mm_MidHeight_Choc_Hotswap_rev5
- SW38: renamed from SW37; footprint MX_Alps_Hybrid:MX-Alps-Hybrid-1.25U -> colbully:CherryMX_18mm_MidHeight_Choc_Hotswap_rev5
- SW39, SW44: footprint MX_Alps_Hybrid:MX-Alps-Hybrid-1.25U -> colbully:CherryMX_18mm_MidHeight_Choc_Hotswap_rev5
- SW40: renamed from SW38; footprint MX_Alps_Hybrid:MX-Alps-Hybrid-1.5U -> colbully:CherryMX_18mm_MidHeight_Choc_Hotswap_rev5
- SW41: renamed from SW39; footprint MX_Alps_Hybrid:MX-Alps-Hybrid-1.25U -> colbully:CherryMX_18mm_MidHeight_Choc_Hotswap_rev5
- SW42: renamed from SW40; footprint MX_Alps_Hybrid:MX-Alps-Hybrid-1.5U -> colbully:CherryMX_18mm_MidHeight_Choc_Hotswap_rev5
- SW43: renamed from SW41; footprint MX_Alps_Hybrid:MX-Alps-Hybrid-2.25U-ReversedStabilizers -> colbully:CherryMX_18mm_MidHeight_Choc_Hotswap_rev5
- SW45: renamed from SW42; footprint MX_Alps_Hybrid:MX-Alps-Hybrid-2.75U-ReversedStabilizers -> colbully:CherryMX_18mm_MidHeight_Choc_Hotswap_rev5
- SW47: renamed from SW43; footprint MX_Alps_Hybrid:MX-Alps-Hybrid-1.5U -> colbully:CherryMX_18mm_MidHeight_Choc_Hotswap_rev5
- SW48: renamed from SW44; footprint MX_Alps_Hybrid:MX-Alps-Hybrid-1.25U -> colbully:CherryMX_18mm_MidHeight_Choc_Hotswap_rev5
- SW49: renamed from SW45; footprint MX_Alps_Hybrid:MX-Alps-Hybrid-1.5U -> colbully:CherryMX_18mm_MidHeight_Choc_Hotswap_rev5
- renumbered D26 to D27, D27 to D28, D28 to D29, D29 to D30, D30 to D31, D31 to D32, D32 to D33, D33 to D34, D34 to D35, D35 to D36, D36 to D37, D37 to D38, D38 to D40, D39 to D41, D40 to D42, D41 to D43, D42 to D45, D43 to D49, D44 to D50, D45 to D51
Connections:
- net CAPS_LED: now also D47.2 (DIN)
- net COL10: now also SW47.1; no longer SW47.2
- net COL11: now also SW48.1; no longer SW44.1, SW48.2
- net COL12: now also SW12.1; no longer SW12.2
- net COL13: now also SW39.1, SW26.1, SW50.1
- net COL2: now also SW41.1; no longer SW39.1, SW41.2
- net COL3: now also SW42.1; no longer SW42.2
- net COL5: now also SW44.1
- net COL8: now also SW45.1; no longer SW45.2
- net COL9: now also SW46.1
- net GND: now also D47.1 (VSS)
- net ROW2: now also D26.1 (K)
- net ROW3: now also D39.1 (K)
- net ROW4: now also D44.1 (K), D48.1 (K), D52.1 (K)
- net at D45.2 (A): now also SW45.2; no longer SW45.1
- net at D49.2 (A): now also SW47.2; no longer SW47.1
- net at D42.2 (A): now also SW42.2; no longer SW42.1
- net at D12.2 (A): now also SW12.2; no longer SW12.1
- net col12_row3_diode: no longer names the net of D38.2 (A), SW38.2
- net col13_row1_diode: no longer names the net of D13.2 (A), SW13.2
- net col1_row2_diode: no longer names the net of D14.2 (A), SW14.2
- new net: D48.2 (A), SW46.2
- new net: D41.2 (A), SW41.2
- new net: D39.2 (A), SW39.2
- new net: D52.2 (A), SW50.2
- new net: D26.2 (A), SW26.2
- new net: D44.2 (A), SW44.2
- new net: D50.2 (A), SW48.2
- new net +5V: D47.3 (VDD)
- no-connect marks 0 -> 1
Other:
- note removed: "2.25u right shift option"
- note removed: "2u backspace option"
- note removed: "indicator led position options"
- note removed: "rotary encoder"
- note removed: "stepped 1.75u option"
- moved on the sheet: D40, D41, D43, D49, D50, D51, SW40, SW41, SW42, SW43, SW45, SW47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

Commit message: Modified top plate model.
Other:
- company: sporkus -> ihsinoky
- title: Bully2040 -> Col-bully2040
Changed lines of the file:
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@@
 	(paper "A4")
 	(title_block
-		(title "Bully2040")
+		(title "Col-bully2040")
 		(date "2023-06-23")
-		(rev "0.2")
-		(company "sporkus")
+		(rev "0.1")
+		(company "ihsinoky")
 		(comment 1 "adding alps and layout options")
 	)
